File: pcb/scot-controller.kicad_pcb (KiCad board)
At the start: 2 copper layers, 55.9 x 52.3 mm, 19 parts, among them IC1 MCP2562, J1 Conn_01x02_Female, J2 Conn_01x03_Female, J3 Conn_01x03_Female, U1 MCP1703A-5002_SOT223, U2 TSR_1-2465

Commit message: pcb: Fix TXD/RXD mapping, move CAN regulator closer, add gitignore.
Parts:
- C4: value 10u/6.5V -> 4u7/6.5V
- C8: value 2u2/5V -> 4u7/5V
- FB1: value Ferrite_Bead_Small -> 600R@100M/1A
- R1: value R -> 120R
- moved U1 12.5 mm to (205.4, 94.6), turned to 180 degrees
- moved C3 9.93 mm to (210.6, 96.2), turned to 90 degrees
- moved C5 5.55 mm to (210.6, 92.9), turned to 270 degrees
Connections:
- A2 pad 31: /CAN_TXD -> /CAN_RXD
- A2 pad 32: /CAN_RXD -> /CAN_TXD
Routing:
- net GND: track 144.9 -> 128.2 mm
- net /6.5VDC: track 36.9 -> 44.8 mm
- net /3V3_HOST: track 59.0 -> 51.2 mm
- net /5V_CAN: track 17.3 -> 12.0 mm
- net /CAN_TXD: track 31.9 -> 35.2 mm
- net /CAN_RXD: track 32.0 -> 29.1 mm, vias 0 -> 1
Other:
- board text added: "May 2020"
- board text removed: "April 2020"
